File: pcb/DIU_hour.kicad_sch (KiCad schematic)
At the start: 6 parts, among them U4 74HC595, U5 74HC595, U6 74HC595

Commit message: Partlist refactoring
Parts:
- C10, C8, C9: Hersteller HTL -> (none); Nummer 100128 -> (none); Vendor (none) -> HTL; VendorId (none) -> 100128
- U4, U5, U6: Hersteller DigiKey -> (none); Nummer 296-26485-1-ND -> (none); Vendor (none) -> HTL; VendorId (none) -> 103445
Changed lines of the file:
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@@
       (effects (font (size 1.27 1.27)) hide)
     )
-    (property "Hersteller" "DigiKey" (at 179.07 76.2 0)
-      (effects (font (size 1.27 1.27)) hide)
-    )
-    (property "Nummer" "296-26485-1-ND" (at 179.07 76.2 0)
+    (property "Vendor" "HTL" (at 179.07 76.2 0)
+      (effects (font (size 1.27 1.27)) hide)
+    )
+    (property "VendorId" "103445" (at 179.07 76.2 0)
       (effects (font (size 1.27 1.27)) hide)
     )
@@
       (effects (font (size 1.27 1.27)) hide)
     )
-    (property "Hersteller" "DigiKey" (at 92.71 76.2 0)
-      (effects (font (size 1.27 1.27)) hide)
-    )
-    (property "Nummer" "296-26485-1-ND" (at 92.71 76.2 0)
+    (property "Vendor" "HTL" (at 92.71 76.2 0)
+      (effects (font (size 1.27 1.27)) hide)
+    )
+    (property "VendorId" "103445" (at 92.71 76.2 0)
       (effects (font (size 1.27 1.27)) hide)
     )
@@
       (effects (font (size 1.27 1.27)) hide)
     )
-    (property "Hersteller" "HTL" (at 76.2 171.45 0)
-      (effects (font (size 1.27 1.27)) hide)
-    )
-    (property "Nummer" "100128" (at 76.2 171.45 0)
+    (property "Vendor" "HTL" (at 76.2 171.45 0)
+      (effects (font (size 1.27 1.27)) hide)
+    )
+    (property "VendorId" "100128" (at 76.2 171.45 0)
       (effects (font (size 1.27 1.27)) hide)
     )
@@
       (effects (font (size 1.27 1.27)) hide)
     )
-    (property "Hersteller" "HTL" (at 63.5 171.45 0)
-      (effects (font (size 1.27 1.27)) hide)
-    )
-    (property "Nummer" "100128" (at 63.5 171.45 0)
+    (property "Vendor" "HTL" (at 63.5 171.45 0)
+      (effects (font (size 1.27 1.27)) hide)
+    )
+    (property "VendorId" "100128" (at 63.5 171.45 0)
       (effects (font (size 1.27 1.27)) hide)
     )
@@
       (effects (font (size 1.27 1.27)) hide)
     )
-    (property "Hersteller" "DigiKey" (at 135.89 76.2 0)
-      (effects (font (size 1.27 1.27)) hide)
-    )
-    (property "Nummer" "296-26485-1-ND" (at 135.89 76.2 0)
+    (property "Vendor" "HTL" (at 135.89 76.2 0)
+      (effects (font (size 1.27 1.27)) hide)
+    )
+    (property "VendorId" "103445" (at 135.89 76.2 0)
       (effects (font (size 1.27 1.27)) hide)
     )
@@
       (effects (font (size 1.27 1.27)) hide)
     )
-    (property "Hersteller" "HTL" (at 50.8 171.45 0)
-      (effects (font (size 1.27 1.27)) hide)
-    )
-    (property "Nummer" "100128" (at 50.8 171.45 0)
-      (effects (font (size 1.27 1.27)) hide)
-    )
+    (property "Vendor" "HTL" (at 50.8 171.45 0)
+      (effects (font (size 1.27 1.27)) hide)
+    )
+    (property "VendorId" "100128" (at 50.8 171.45 0)
+      (effects (font (size 1.27 1.27)) hide)
+    )
