File: pcb/DIU_visual.kicad_sch (KiCad schematic)
At the start: 176 parts, among them J10 Conn_01x21_Pin, J11 Conn_01x21_Socket, J12 Conn_01x21_Socket, J13 Conn_01x21_Pin, J6 Conn_01x21_Pin, J7 Conn_01x21_Socket, J8 Conn_01x21_Pin, J9 Conn_01x21_Socket

Commit message: Partlist refactoring
Parts:
- D1, D10, D11, D12, D13, D14, D15, D16, D17, D18, D19, D2, D20, D21, D22, D23, D24, D25, D26, D27, D28, D29, D3, D30, D31, D32, D33, D34, D35, D36, D37, D38, D39, D4, D40, D41, D42, D43, D44, D45, D46, D47, D48, D49, D5, D50, D51, D52, D53, D54, D55, D56, D57, D58, D59, D6, D60, D61, D62, D63, D64, D65, D66, D67, D68, D69, D7, D70, D71, D72, D73, D74, D75, D76, D77, D78, D79, D8, D80, D81, D82, D83, D84, D9: Hersteller DigiKey -> (none); Nummer 1830-1090-2-ND -> (none); Vendor (none) -> HTL; VendorId (none) -> 103437
- J10, J13, J6, J8: Hersteller HTL -> (none); Nummer 101521 -> (none); Vendor (none) -> HTL; VendorId (none) -> 101521
- J11, J12, J7, J9: Hersteller HTL -> (none); Nummer 101546 -> (none); Vendor (none) -> HTL; VendorId (none) -> 101546
- R1, R10, R11, R12, R13, R14, R15, R16, R17, R18, R19, R2, R20, R21, R22, R23, R24, R25, R26, R27, R28, R29, R3, R30, R31, R32, R33, R34, R35, R36, R37, R38, R39, R4, R40, R41, R42, R43, R44, R45, R46, R47, R48, R49, R5, R50, R51, R52, R53, R54, R55, R56, R57, R58, R59, R6, R60, R61, R62, R63, R64, R65, R66, R67, R68, R69, R7, R70, R71, R72, R73, R74, R75, R76, R77, R78, R79, R8, R80, R81, R82, R83, R84, R9: Hersteller HTL -> (none); Nummer 102930 -> (none); Vendor (none) -> HTL; VendorId (none) -> 102930
