File: pcb/DIU.kicad_pcb (KiCad board)
At the start: 2 copper layers, 143.5 x 68.6 mm, 272 parts, among them J1 Conn_01x02_Pin, J10 Conn_01x21_Pin, J11 Conn_01x21_Socket, J12 Conn_01x21_Socket, J13 Conn_01x21_Pin, J14 Conn_01x01_Socket, J15 Conn_01x01_Pin, J16 Conn_01x01_Pin, J17 Conn_01x01_Socket, J18 Battery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

Commit message: Change reset circuit
Parts:
- removed R96: n.B., Resistor_SMD:R_0603_1608Metric
- added C11: 10u, Capacitor_SMD:C_0603_1608Metric, F.Cu at (218.8, 113.2)
