File: pcb/DIU.kicad_pcb (KiCad board)
At the start: 2 copper layers, 143.5 x 68.6 mm, 272 parts, among them J1 Conn_01x02_Pin, J10 Conn_01x21_Pin, J11 Conn_01x21_Socket, J12 Conn_01x21_Socket, J13 Conn_01x21_Pin, J14 Conn_01x01_Socket, J15 Conn_01x01_Pin, J16 Conn_01x01_Pin, J17 Conn_01x01_Socket, J18 Battery, J2 Conn_01x02_Pin, J3 Conn_01x03_Pin, J4 USB_OTG, J5 Conn_01x03_Socket, J6 Conn_01x21_Pin, J7 Conn_01x21_Socket, J8 Conn_01x21_Pin, J9 Conn_01x21_Socket, Q1 2N7002E, SW1 SW_SPST, SW2 SW_SPST, SW3 SW_SPST, SW4 SW_SPST, U1 LD1117S33TR, U10 74HC595, U11 74HC595, U12 74HC595, U13 74HC595, U14 74HC595, U15 MCP7940N-xMS, U2 FT232RL, U3 ATtiny1606-S, U4 74HC595, U5 74HC595, U6 74HC595, U7 74HC595, U8 74HC595, U9 74HC595, Y1 32.768kHz

Commit message: Add resistor to reset circuit
Parts:
- R95: value n.B. -> 330k
Changed lines of the file:
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@@
     (property "Sheetname" "")
     (property "Vendor" "HTL")
-    (property "VendorId" "")
+    (property "VendorId" "103238")
     (property "ki_description" "Resistor")
     (property "ki_keywords" "R res resistor")
@@
         (effects (font (size 0.75 0.75) (thickness 0.12)))
     )
-    (fp_text value "n.B." (at 0 -1.397) (layer "F.Fab")
+    (fp_text value "330k" (at 0 -1.397) (layer "F.Fab")
         (effects (font (size 1 1) (thickness 0.15)))
     )
