File: pcb/DIU.kicad_pcb (KiCad board)
At the start: 2 copper layers, 143.5 x 68.6 mm, 272 parts, among them J1 Conn_01x02_Pin, J10 Conn_01x21_Pin, J11 Conn_01x21_Socket, J12 Conn_01x21_Socket, J13 Conn_01x21_Pin, J14 Conn_01x01_Socket, J15 Conn_01x01_Pin, J16 Conn_01x01_Pin, J17 Conn_01x01_Socket, J18 Battery, J2 Conn_01x02_Pin, J3 Conn_01x03_Pin, J4 USB_OTG, J5 Conn_01x03_Socket, J6 Conn_01x21_Pin, J7 Conn_01x21_Socket, J8 Conn_01x21_Pin, J9 Conn_01x21_Socket, Q1 2N7002E, SW1 SW_SPST, SW2 SW_SPST, SW3 SW_SPST, SW4 SW_SPST, U1 LD1117S33TR, U10 74HC595, U11 74HC595, U12 74HC595, U13 74HC595, U14 74HC595, U15 MCP7940N-xMS, U2 FT232RL, U3 ATtiny1606-S, U4 74HC595, U5 74HC595, U6 74HC595, U7 74HC595, U8 74HC595, U9 74HC595, Y1 32.768kHz

Commit message: Fix wrong led polarity
Parts:
- turned D89 to 90 degrees
- turned D90 to -90 degrees
Connections:
- R92 pad 1: Net-(D89-K) -> Net-(D89-A)
- R93 pad 1: Net-(D90-K) -> Net-(D90-A)
- U2 pad 22: Net-(D89-A) -> Net-(D89-K)
- U2 pad 23: Net-(D90-A) -> Net-(D90-K)
Routing:
- net Net-(D90-K): track 2.09 -> 9.87 mm, vias 0 -> 1
- net Net-(D90-A): track 9.87 -> 2.09 mm, vias 1 -> 0
- net Net-(D89-K): track 2.25 -> 9.40 mm, vias 0 -> 1
- net Net-(D89-A): track 9.40 -> 2.25 mm, vias 1 -> 0
Changed lines of the file:
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@@
       (net 3 "GND") (pinfunction "GND") (pintype "power_in"))
     (pad "22" smd rect (at 3.6 -0.325) (size 1.75 0.45) (layers "F.Cu" "F.Paste" "F.Mask")
-      (net 184 "Net-(D89-A)") (pinfunction "CBUS1") (pintype "bidirectional"))
+      (net 183 "Net-(D89-K)") (pinfunction "CBUS1") (pintype "bidirectional"))
     (pad "23" smd rect (at 3.6 -0.975) (size 1.75 0.45) (layers "F.Cu" "F.Paste" "F.Mask")
-      (net 186 "Net-(D90-A)") (pinfunction "CBUS0") (pintype "bidirectional"))
+      (net 185 "Net-(D90-K)") (pinfunction "CBUS0") (pintype "bidirectional"))
     (pad "24" smd rect (at 3.6 -1.625) (size 1.75 0.45) (layers "F.Cu" "F.Paste" "F.Mask"))
     (pad "25" smd rect (at 3.6 -2.275) (size 1.75 0.45) (layers "F.Cu" "F.Paste" "F.Mask")
@@
   )
   (footprint "LED_SMD:LED_0603_1608Metric" (layer "B.Cu")
-    (at 225.425 100.33 90)
+    (at 225.425 100.33 -90)
     (descr "LED SMD 0603 (1608 Metric), square (rectangular) end terminal, IPC_7351 nominal, (Body size source: http://www.tortai-tech.com/upload/download/2011102023233369053.pdf), generated with kicad-footprint-generator")
     (tags "LED")
@@
     (property "ki_keywords" "LED diode")
     (attr smd)
-    (fp_text reference "D90" (at 0 -2.286 90) (layer "B.SilkS")
+    (fp_text reference "D90" (at 0.254 -1.397 90) (layer "B.SilkS")
         (effects (font (size 0.75 0.75) (thickness 0.12)) (justify mirror))
     )
@@
     (fp_line (start 0.8 0.4) (end -0.5 0.4)
       (stroke (width 0.1) (type solid)) (layer "B.Fab"))
-    (pad "1" smd roundrect (at -0.7875 0 90) (size 0.875 0.95) (layers "B.Cu" "B.Paste" "B.Mask") (roundrect_rratio 0.25)
+    (pad "1" smd roundrect (at -0.7875 0 270) (size 0.875 0.95) (layers "B.Cu" "B.Paste" "B.Mask") (roundrect_rratio 0.25)
       (net 185 "Net-(D90-K)") (pinfunction "K") (pintype "passive"))
-    (pad "2" smd roundrect (at 0.7875 0 90) (size 0.875 0.95) (layers "B.Cu" "B.Paste" "B.Mask") (roundrect_rratio 0.25)
+    (pad "2" smd roundrect (at 0.7875 0 270) (size 0.875 0.95) (layers "B.Cu" "B.Paste" "B.Mask") (roundrect_rratio 0.25)
       (net 186 "Net-(D90-A)") (pinfunction "A") (pintype "passive"))
     (model "${KICAD6_3DMODEL_DIR}/LED_SMD.3dshapes/LED_0603_1608Metric.wrl"
@@
       (stroke (width 0.1) (type solid)) (layer "B.Fab"))
     (pad "1" smd roundrect (at -0.825 0 180) (size 0.8 0.95) (layers "B.Cu" "B.Paste" "B.Mask") (roundrect_rratio 0.25)
-      (net 185 "Net-(D90-K)") (pintype "passive"))
+      (net 186 "Net-(D90-A)") (pintype "passive"))
     (pad "2" smd roundrect (at 0.825 0 180) (size 0.8 0.95) (layers "B.Cu" "B.Paste" "B.Mask") (roundrect_rratio 0.25)
       (net 4 "VBUS") (pintype "passive"))
@@
   )
   (footprint "LED_SMD:LED_0603_1608Metric" (layer "B.Cu")
-    (at 225.425 107.4675 -90)
+    (at 225.425 107.4675 90)
     (descr "LED SMD 0603 (1608 Metric), square (rectangular) end terminal, IPC_7351 nominal, (Body size source: http://www.tortai-tech.com/upload/download/2011102023233369053.pdf), generated with kicad-footprint-generator")
     (tags "LED")
@@
     (property "ki_keywords" "LED diode")
     (attr smd)
-    (fp_text reference "D89" (at 3.5305 -0.889 -90) (layer "B.SilkS")
+    (fp_text reference "D89" (at -1.4985 1.397 90) (layer "B.SilkS")
         (effects (font (size 0.75 0.75) (thickness 0.12)) (justify mirror))
     )
-    (fp_text value "LED" (at 0 -1.43 90) (layer "B.Fab")
+    (fp_text value "LED" (at 0 1.397 90) (layer "B.Fab")
         (effects (font (size 1 1) (thickness 0.15)) (justify mirror))
     )
@@
     (fp_line (start 0.8 0.4) (end -0.5 0.4)
       (stroke (width 0.1) (type solid)) (layer "B.Fab"))
-    (pad "1" smd roundrect (at -0.7875 0 270) (size 0.875 0.95) (layers "B.Cu" "B.Paste" "B.Mask") (roundrect_rratio 0.25)
+    (pad "1" smd roundrect (at -0.7875 0 90) (size 0.875 0.95) (layers "B.Cu" "B.Paste" "B.Mask") (roundrect_rratio 0.25)
       (net 183 "Net-(D89-K)") (pinfunction "K") (pintype "passive"))
-    (pad "2" smd roundrect (at 0.7875 0 270) (size 0.875 0.95) (layers "B.Cu" "B.Paste" "B.Mask") (roundrect_rratio 0.25)
+    (pad "2" smd roundrect (at 0.7875 0 90) (size 0.875 0.95) (layers "B.Cu" "B.Paste" "B.Mask") (roundrect_rratio 0.25)
       (net 184 "Net-(D89-A)") (pinfunction "A") (pintype "passive"))
     (model "${KICAD6_3DMODEL_DIR}/LED_SMD.3dshapes/LED_0603_1608Metric.wrl"
@@
       (stroke (width 0.1) (type solid)) (layer "B.Fab"))
     (pad "1" smd roundrect (at -0.825 0 180) (size 0.8 0.95) (layers "B.Cu" "B.Paste" "B.Mask") (roundrect_rratio 0.25)
-      (net 183 "Net-(D89-K)") (pintype "passive"))
+      (net 184 "Net-(D89-A)") (pintype "passive"))
     (pad "2" smd roundrect (at 0.825 0 180) (size 0.8 0.95) (layers "B.Cu" "B.Paste" "B.Mask") (roundrect_rratio 0.25)
       (net 4 "VBUS") (pintype "passive"))
@@
   (segment (start 176.53 99.32) (end 176.53 98.1965) (width 0.3) (layer "B.Cu") (net 182))
   (segment (start 176.53 98.1965) (end 177.165 97.5615) (width 0.3) (layer "B.Cu") (net 182))
-  (segment (start 225.425 105.6) (end 226.25 104.775) (width 0.3) (layer "B.Cu") (net 183))
-  (segment (start 225.425 106.68) (end 225.425 105.6) (width 0.3) (layer "B.Cu") (net 183))
-  (segment (start 223.957 104.577) (end 225.425 106.045) (width 0.3) (layer "F.Cu") (net 184))
-  (segment (start 225.425 106.045) (end 225.425 109.217894) (width 0.3) (layer "F.Cu") (net 184))
-  (segment (start 225.426053 109.218947) (end 225.425 109.217894) (width 0.3) (layer "F.Cu") (net 184))
-  (segment (start 220.77 104.577) (end 223.957 104.577) (width 0.3) (layer "F.Cu") (net 184))
-  (via (at 225.425 109.217894) (size 0.4) (drill 0.3) (layers "F.Cu" "B.Cu") (net 184))
-  (segment (start 225.425 109.217894) (end 225.425 108.255) (width 0.3) (layer "B.Cu") (net 184))
-  (segment (start 225.425 101.1175) (end 225.425 102.045) (width 0.3) (layer "B.Cu") (net 185))
-  (segment (start 225.425 102.045) (end 226.25 102.87) (width 0.3) (layer "B.Cu") (net 185))
-  (segment (start 224.282 99.5426) (end 225.425 100.6856) (width 0.3) (layer "F.Cu") (net 186))
-  (segment (start 225.425 100.6856) (end 225.425 102.590456) (width 0.3) (layer "F.Cu") (net 186))
-  (segment (start 225.425 102.590456) (end 224.088456 103.927) (width 0.3) (layer "F.Cu") (net 186))
-  (segment (start 224.088456 103.927) (end 220.77 103.927) (width 0.3) (layer "F.Cu") (net 186))
-  (via (at 224.282 99.5426) (size 0.4) (drill 0.3) (layers "F.Cu" "B.Cu") (net 186))
-  (segment (start 224.2821 99.5425) (end 225.425 99.5425) (width 0.3) (layer "B.Cu") (net 186))
-  (segment (start 224.282 99.5426) (end 224.2821 99.5425) (width 0.3) (layer "B.Cu") (net 186))
+  (segment (start 223.957 104.577) (end 225.425 106.045) (width 0.3) (layer "F.Cu") (net 183))
+  (segment (start 225.425 106.045) (end 225.425 109.217894) (width 0.3) (layer "F.Cu") (net 183))
+  (segment (start 225.426053 109.218947) (end 225.425 109.217894) (width 0.3) (layer "F.Cu") (net 183))
+  (segment (start 220.77 104.577) (end 223.957 104.577) (width 0.3) (layer "F.Cu") (net 183))
+  (via (at 225.425 109.217894) (size 0.4) (drill 0.3) (layers "F.Cu" "B.Cu") (net 183))
+  (segment (start 225.425 109.217894) (end 225.425 108.255) (width 0.3) (layer "B.Cu") (net 183))
+  (segment (start 225.425 105.6) (end 226.25 104.775) (width 0.3) (layer "B.Cu") (net 184))
+  (segment (start 225.425 106.68) (end 225.425 105.6) (width 0.3) (layer "B.Cu") (net 184))
+  (segment (start 224.282 99.5426) (end 225.425 100.6856) (width 0.3) (layer "F.Cu") (net 185))
+  (segment (start 225.425 100.6856) (end 225.425 102.590456) (width 0.3) (layer "F.Cu") (net 185))
+  (segment (start 225.425 102.590456) (end 224.088456 103.927) (width 0.3) (layer "F.Cu") (net 185))
+  (segment (start 224.088456 103.927) (end 220.77 103.927) (width 0.3) (layer "F.Cu") (net 185))
+  (via (at 224.282 99.5426) (size 0.4) (drill 0.3) (layers "F.Cu" "B.Cu") (net 185))
+  (segment (start 224.2821 99.5425) (end 225.425 99.5425) (width 0.3) (layer "B.Cu") (net 185))
+  (segment (start 224.282 99.5426) (end 224.2821 99.5425) (width 0.3) (layer "B.Cu") (net 185))
+  (segment (start 225.425 101.1175) (end 225.425 102.045) (width 0.3) (layer "B.Cu") (net 186))
+  (segment (start 225.425 102.045) (end 226.25 102.87) (width 0.3) (layer "B.Cu") (net 186))
   (segment (start 200.909 114.93) (end 200.914 114.935) (width 1) (layer "F.Cu") (net 187))
   (segment (start 200.909 112.395) (end 200.909 114.93) (width 1) (layer "F.Cu") (net 187))
