File: pcb/DIU_minute.kicad_sch (KiCad schematic)
At the start: 28 parts, among them J14 Conn_01x01_Socket, J15 Conn_01x01_Pin, J16 Conn_01x01_Pin, J17 Conn_01x01_Socket, U10 74HC595, U11 74HC595, U12 74HC595, U13 74HC595, U14 74HC595, U7 74HC595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

Commit message: Partlist refactoring
Parts:
- C18, C19, C20, C21, C23, C25, C27, C29: Hersteller HTL -> (none); Nummer 100128 -> (none); Vendor (none) -> HTL; VendorId (none) -> 100128
- D85, D86, D87, D88: Hersteller DigiKey -> (none); Nummer 160-1830-1-ND, 160-1828-1-ND, 4 x 160-1827-1-ND -> (none); Vendor (none) -> HTL; VendorId (none) -> 103438, 103439, 4 x 103440
- J14, J17: Hersteller HTL -> (none); Nummer 101546 -> (none); Vendor (none) -> HTL; VendorId (none) -> 101546
- J15, J16: Hersteller HTL -> (none); Nummer 101521 -> (none); Vendor (none) -> HTL; VendorId (none) -> 101521
- R85, R86, R87, R88: Hersteller HTL -> (none); Nummer 103164 -> (none); Vendor (none) -> HTL; VendorId (none) -> 103164
- U10, U11, U12, U13, U14, U7, U8, U9: Hersteller DigiKey -> (none); Nummer 296-26485-1-ND -> (none); Vendor (none) -> HTL; VendorId (none) -> 103445

Commit message: Adapt vendor-ids on leds
Parts:
- D85: VendorId 103438, 103439, 4 x 103440 -> 103438
- D86, D87: VendorId 103438, 103439, 4 x 103440 -> 103440
- D88: VendorId 103438, 103439, 4 x 103440 -> 103439
Changed lines of the file:
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@@
       (effects (font (size 1.27 1.27)) hide)
     )
-    (property "VendorId" "103438, 103439, 4 x 103440" (at 163.83 165.1 0)
+    (property "VendorId" "103439" (at 163.83 165.1 0)
       (effects (font (size 1.27 1.27)) hide)
     )
@@
       (effects (font (size 1.27 1.27)) hide)
     )
-    (property "VendorId" "103438, 103439, 4 x 103440" (at 153.67 165.1 0)
+    (property "VendorId" "103440" (at 153.67 165.1 0)
       (effects (font (size 1.27 1.27)) hide)
     )
@@
       (effects (font (size 1.27 1.27)) hide)
     )
-    (property "VendorId" "103438, 103439, 4 x 103440" (at 158.75 165.1 0)
+    (property "VendorId" "103440" (at 158.75 165.1 0)
       (effects (font (size 1.27 1.27)) hide)
     )
@@
       (effects (font (size 1.27 1.27)) hide)
     )
-    (property "VendorId" "103438, 103439, 4 x 103440" (at 148.59 165.1 0)
-      (effects (font (size 1.27 1.27)) hide)
-    )
+    (property "VendorId" "103438" (at 148.59 165.1 0)
+      (effects (font (size 1.27 1.27)) hide)
+    )
